File: Sonar/main.sch (EAGLE design)
At the start: 10 parts, among them IC1 4066N, Q1 BC488

Commit message: Minor layout changes.
Parts:
- removed SV1, SV2, SV3: (no value), con-lstb:MA03-1
- added J1: (no value), jumper:JUMPER
- added JP1: (no value), pinhead:PINHD-1X2
- added JP3: (no value), pinhead:PINHD-1X5
- added JP4: (no value), jumper:JP2E
- C1: value (none) -> 100n
- C2: value (none) -> 220n
- C3: value (none) -> 100u
- R1: value (none) -> 470R
- R2: value (none) -> 2k2
Connections:
- removed net N$1: IC1A.C, Q1.B, R2.2, SV3.2
- removed net N$2: IC1A.B, SV3.1
- new net N$8: IC1A.C, JP4.2
- new net OUT: IC1A.B, JP3.1
- new net OUT-ENABLE: JP3.3, JP4.1
- new net SPEAKER-IN: JP3.2, JP4.3, Q1.B, R2.2
- net GND: now also JP3.5; no longer SV2.2, SV2.3, SV3.3
- net N$3: now also JP1.2; no longer SV1.1, SV1.2
- net VCC: now also JP1.1, JP3.4; no longer SV1.3, SV2.1
Other:
- moved on the sheet: C1, C2, C3, IC1A, IC1P, R1
